File: 23LC1024_pcb/23LC1024_pcb.kicad_sch (KiCad schematic)
At the start: 9 parts, among them J1 Conn_01x06_Male_JA, J2 Conn_01x06_Male_JB, U1 23LC1024-I/P, U2 AP2141SG-13

Commit message: 23LC1024 PCB: Assign footprints, create schematic
Parts:
- C1, C2, C3, C4: footprint (none) -> Capacitor_SMD:C_1206_3216Metric_Pad1.33x1.80mm_HandSolder
Changed lines of the file:
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@@
       (effects (font (size 1.27 1.27)) (justify left))
     )
-    (property "Footprint" "" (id 2) (at 115.2652 41.91 0)
+    (property "Footprint" "Capacitor_SMD:C_1206_3216Metric_Pad1.33x1.80mm_HandSolder" (id 2) (at 115.2652 41.91 0)
       (effects (font (size 1.27 1.27)) hide)
     )
@@
       (effects (font (size 1.27 1.27)) (justify right))
     )
-    (property "Footprint" "" (id 2) (at 127.3048 34.29 0)
+    (property "Footprint" "Capacitor_SMD:C_1206_3216Metric_Pad1.33x1.80mm_HandSolder" (id 2) (at 127.3048 34.29 0)
       (effects (font (size 1.27 1.27)) hide)
     )
@@
       (effects (font (size 1.27 1.27)) (justify right))
     )
-    (property "Footprint" "" (id 2) (at 62.5348 78.74 0)
+    (property "Footprint" "Capacitor_SMD:C_1206_3216Metric_Pad1.33x1.80mm_HandSolder" (id 2) (at 62.5348 78.74 0)
       (effects (font (size 1.27 1.27)) hide)
     )
@@
       (effects (font (size 1.27 1.27)) (justify left))
     )
-    (property "Footprint" "" (id 2) (at 58.1152 86.36 0)
+    (property "Footprint" "Capacitor_SMD:C_1206_3216Metric_Pad1.33x1.80mm_HandSolder" (id 2) (at 58.1152 86.36 0)
       (effects (font (size 1.27 1.27)) hide)
     )
@@
     )
     (path "/f5f140cb-6fcf-46b3-9c75-481fb0c82d9c"
-      (reference "C1") (unit 1) (value "120 uF") (footprint "")
+      (reference "C1") (unit 1) (value "120 uF") (footprint "Capacitor_SMD:C_1206_3216Metric_Pad1.33x1.80mm_HandSolder")
     )
     (path "/df8fa7ea-1025-4e61-86fc-128ea1388b0a"
-      (reference "C2") (unit 1) (value "0.1 uF") (footprint "")
+      (reference "C2") (unit 1) (value "0.1 uF") (footprint "Capacitor_SMD:C_1206_3216Metric_Pad1.33x1.80mm_HandSolder")
     )
     (path "/2457f839-055e-4272-9d36-aa5684e80891"
-      (reference "C3") (unit 1) (value "0.1 uF") (footprint "")
+      (reference "C3") (unit 1) (value "0.1 uF") (footprint "Capacitor_SMD:C_1206_3216Metric_Pad1.33x1.80mm_HandSolder")
     )
     (path "/cdc87dac-c079-4199-8e8f-f38b4ba2c177"
-      (reference "C4") (unit 1) (value "120 uF") (footprint "")
+      (reference "C4") (unit 1) (value "120 uF") (footprint "Capacitor_SMD:C_1206_3216Metric_Pad1.33x1.80mm_HandSolder")
     )
     (path "/faad28a2-09fa-4ce9-a367-71b6860b94ed"
-      (reference "J1") (unit 1) (value "Conn_01x06_Male_JA") (footprint "")
+      (reference "J1") (unit 1) (value "Conn_01x06_Male_JA") (footprint "Connector_PinHeader_2.54mm:PinHeader_1x06_P2.54mm_Horizontal")
     )
     (path "/8eb98c56-17e4-4de6-a3e3-06dcfa392040"
-      (reference "J2") (unit 1) (value "Conn_01x06_Male_JB") (footprint "")
+      (reference "J2") (unit 1) (value "Conn_01x06_Male_JB") (footprint "Connector_PinHeader_2.54mm:PinHeader_1x06_P2.54mm_Horizontal")
     )
     (path "/93a291ff-b4f5-47f6-8bbe-1414f52b4524"
-      (reference "R1") (unit 1) (value "10 K") (footprint "")
+      (reference "R1") (unit 1) (value "10 K") (footprint "Resistor_SMD:R_1206_3216Metric_Pad1.30x1.75mm_HandSolder")
     )
     (path "/580b6ef9-391f-432e-b992-da972344253f"

Commit message: 23LC1024 PCB: Finish routing
Parts:
- removed C1, C4: 120 uF, Capacitor_SMD:C_1206_3216Metric_Pad1.33x1.80mm_HandSolder, symbol Device:C_Polarized
- J1, J2: footprint (none) -> Connector_PinHeader_2.54mm:PinHeader_1x06_P2.54mm_Horizontal
- R1: footprint (none) -> Resistor_SMD:R_1206_3216Metric_Pad1.30x1.75mm_HandSolder
- renumbered C2 to C1, C3 to C2
Connections:
- net +3V3: no longer C1.2, J1.6 (3V3), J2.6 (3V3), R1.2, U2.2 (IN), U2.3 (IN)
- net CLK: now also J2.6 (CLK); no longer J2.1 (CLK)
- net CS: now also J2.4 (CS); no longer J2.3 (CS)
- net EN: now also J2.3 (EN); no longer J2.4 (EN)
- net FLG: now also J2.5 (FLG); no longer J2.2 (FLG)
- net GND: now also J1.2 (GND), J2.2 (GND); no longer J1.5 (GND), J2.5 (GND)
- net SIO0: now also J1.6 (SIO0); no longer J1.1 (SIO0)
- net SIO1: now also J1.5 (SIO1); no longer J1.2 (SIO1)
- net SIO2: now also J1.4 (SIO2); no longer J1.3 (SIO2)
- net SIO3: now also J1.3 (SIO3); no longer J1.4 (SIO3)
- new net BASYS3V3: C1.2, J1.1 (3V3), J2.1 (3V3), R1.2, U2.2 (IN), U2.3 (IN)
Other:
- moved on the sheet: J1, J2

Commit message: 23LC1024 PCB: Rework to add three
Parts:
- removed C1: 0.1 uF, Capacitor_SMD:C_1206_3216Metric_Pad1.33x1.80mm_HandSolder, symbol Device:C
- removed U2: AP2141SG-13, Package_SO:SO-8_3.9x4.9mm_P1.27mm, symbol AP2141SG-13:AP2141SG-13
- added C2, C3: 0.1 uF, Capacitor_SMD:C_1206_3216Metric_Pad1.33x1.80mm_HandSolder, symbol Device:C
- added R2, R3: 10K, Resistor_SMD:R_1206_3216Metric_Pad1.30x1.75mm_HandSolder, symbol Device:R
- added U2, U3: 23LC1024-I/P, Package_DIP:DIP-8_W7.62mm, symbol 23LC1024IP:23LC1024-I/P
- R1: value 10 K -> 10K
- renumbered C2 to C1
Connections:
- net +3V3 is gone; now on net BASYS3V3: C1.2, U1.8 (VCC)
- net EN is gone; now on net CS_1: J2.3 (CS_1)
- net BASYS3V3: now also R1.1, C2.2, C3.2, R2.1, R3.1, U2.8 (VCC), U3.8 (VCC); no longer R1.2
- net CLK: now also U2.6 (SCK), U3.6 (SCK)
- net GND: now also C2.1, C3.1, U2.4 (VSS), U3.4 (VSS)
- net SIO0: now also U2.5 (SI/SIO0), U3.5 (SI/SIO0)
- net SIO1: now also U2.2 (SO/SIO1), U3.2 (SO/SIO1)
- net SIO2: now also U2.3 (SIO2), U3.3 (SIO2)
- net SIO3: now also U2.7 (*HOLD/SIO3), U3.7 (*HOLD/SIO3)
- net CS renamed CS_1
- net CS_1: now also R1.2; no longer J2.4 (CS)
- net FLG renamed CS_3
- net CS_3: now also R3.2, U3.1 (*CS); no longer R1.1
- new net CS_2: J2.4 (CS_2), R2.2, U2.1 (*CS)
